Commit message: containerized version of moveIt with a package to load kr210 urdf file

File: kr210_urdf/src/urdf/kr210l150_remus.urdf (robot description, URDF)
Before this commit: robot remus, 8 links, 7 joints
Links:
- link remus_base_link: geometry collision mesh filename=package://kr210_urdf/meshes/collision/base_link.stl; visual mesh filename=package://kr210_urdf/meshes/visual/base_link.dae
- link remus_link_1: geometry collision mesh filename=package://kr210_urdf/meshes/collision/link_1.stl; visual mesh filename=package://kr210_urdf/meshes/visual/link_1.dae
- link remus_link_2: geometry collision mesh filename=package://kr210_urdf/meshes/collision/link_2.stl; visual mesh filename=package://kr210_urdf/meshes/visual/link_2.dae
- link remus_link_3: geometry collision mesh filename=package://kr210_urdf/meshes/collision/link_3.stl; visual mesh filename=package://kr210_urdf/meshes/visual/link_3.dae
- link remus_link_4: geometry collision mesh filename=package://kr210_urdf/meshes/collision/link_4.stl; visual mesh filename=package://kr210_urdf/meshes/visual/link_4.dae
- link remus_link_5: geometry collision mesh filename=package://kr210_urdf/meshes/collision/link_5.stl; visual mesh filename=package://kr210_urdf/meshes/visual/link_5.dae
- link remus_link_6: geometry collision mesh filename=package://kr210_urdf/meshes/collision/link_6.stl; visual mesh filename=package://kr210_urdf/meshes/visual/link_6.dae
